Commit message: Re structured code so that there is a table urdf located at a fixed offset from the robot's base frame. I used the static frame publisher to publish the frame. I then did some general code clean up. The user can specify where the table is relative to the robot and then define the table's dimension and the camera will filter the volume above the table

File: src/sawyer_ping_pong/urdf/box.urdf (robot description, URDF)
Before this commit: robot simple_box, 1 links, 0 joints
Links:
- removed link my_box
- added link table; visual box size=1.0 1.0 1.0
- added link world
Joints:
- added joint j1: type fixed, parent world, child table, origin xyz=0 0 0 rpy=0 0 0
